File: hardware/peakick/peakick.kicad_pcb (KiCad board)
At the start: 2 copper layers, 58.4 x 54 mm, 36 parts, among them J1 CONN_161X16_SM_SQ_NOSILK, J2 QWIIC_RA, J3 CONN_12SM_SQ_NO_SILK, SW1 JS102011SAQN, U1 BMP390, U2 SAM-M10Q, U3 ICM-42688-P, U4 MMC5983MA, X1 JSTPH

Commit message: Doc updates
Other:
- board text added: "peakick V1 https://github.com/rrainey/tempo Riley Rainey 2023"
- board text removed: "peakick V1 https://github.com/rrainey/peakick Riley Rainey 2023"
Changed lines of the file:
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@@
     (descr "Resistor SMD 0603 (1608 Metric), square (rectangular) end terminal, IPC_7351 nominal, (Body size source: IPC-SM-782 page 72, https://www.pcb-3d.com/wordpress/wp-content/uploads/ipc-sm-782a_amendment_1_and_2.pdf), generated with kicad-footprint-generator")
     (tags "resistor")
-    (property "NOTES" "1%")
+    (property "NOTES" "10%")
     (property "Sheetfile" "peakick.kicad_sch")
     (property "Sheetname" "")
@@
     (descr "Resistor SMD 0603 (1608 Metric), square (rectangular) end terminal, IPC_7351 nominal, (Body size source: IPC-SM-782 page 72, https://www.pcb-3d.com/wordpress/wp-content/uploads/ipc-sm-782a_amendment_1_and_2.pdf), generated with kicad-footprint-generator")
     (tags "resistor")
-    (property "NOTES" "1%")
+    (property "NOTES" "10%")
     (property "Sheetfile" "peakick.kicad_sch")
     (property "Sheetname" "")
@@
     (descr "LED SMD 0603 (1608 Metric), square (rectangular) end terminal, IPC_7351 nominal, (Body size source: http://www.tortai-tech.com/upload/download/2011102023233369053.pdf), generated with kicad-footprint-generator")
     (tags "LED")
+    (property "MANUFACTURER" "Lite-On")
     (property "MPN" "LTST-S270KGKT")
     (property "NOTES" "GREEN LED")
@@
     (descr "Resistor SMD 0603 (1608 Metric), square (rectangular) end terminal, IPC_7351 nominal, (Body size source: IPC-SM-782 page 72, https://www.pcb-3d.com/wordpress/wp-content/uploads/ipc-sm-782a_amendment_1_and_2.pdf), generated with kicad-footprint-generator")
     (tags "resistor")
-    (property "NOTES" "1%")
+    (property "NOTES" "10%")
     (property "Sheetfile" "peakick.kicad_sch")
     (property "Sheetname" "")
@@
     (at 177.809999 105.515001 90)
     (tags "MMC5983MA ")
+    (property "MAXIMUM_PACKAGE_HEIGHT" "1.0mm")
     (property "MPN" "MMC5983MA")
     (property "Sheetfile" "peakick.kicad_sch")
@@
     (descr "Resistor SMD 0603 (1608 Metric), square (rectangular) end terminal, IPC_7351 nominal, (Body size source: IPC-SM-782 page 72, https://www.pcb-3d.com/wordpress/wp-content/uploads/ipc-sm-782a_amendment_1_and_2.pdf), generated with kicad-footprint-generator")
     (tags "resistor")
+    (property "NOTES" "10K if SAM-M10 not installed")
     (property "Sheetfile" "peakick.kicad_sch")
     (property "Sheetname" "")
@@
     (descr "Resistor SMD 0603 (1608 Metric), square (rectangular) end terminal, IPC_7351 nominal, (Body size source: IPC-SM-782 page 72, https://www.pcb-3d.com/wordpress/wp-content/uploads/ipc-sm-782a_amendment_1_and_2.pdf), generated with kicad-footprint-generator")
     (tags "resistor")
+    (property "NOTES" "10K if SAM-M10 not installed")
     (property "Sheetfile" "peakick.kicad_sch")
     (property "Sheetname" "")
@@
     (at 179.22 75.4 180)
     (descr "2-Pin JST PH Series Right-Angle Connector (+/- for batteries)")
+    (property "MPN" "S2B-PH-SM4-TB")
     (property "Manufacturer Part" "S2B-PH-SM4-TB")
     (property "Sheetfile" "peakick.kicad_sch")
@@
     (at 177.56 98.7467 180)
     (descr "<h3>SMD- 4 Pin Right Angle </h3>\n<p>Specifications:\n<ul><li>Pin count:4</li>\n<li>Pin pitch:0.1\"</li>\n</ul></p>\n<p>Example device(s):\n<ul><li>CONN_04</li>\n</ul></p>")
+    (property "NOTES" "DNP")
     (property "Sheetfile" "peakick.kicad_sch")
     (property "Sheetname" "")
@@
   (gr_line (start 139.97 114.75) (end 139.97 116.34)
     (stroke (width 0.1) (type default)) (layer "F.Fab"))
-  (gr_text "peakick V1\n\nhttps://github.com/rrainey/peakick\nRiley Rainey 2023" (at 130.96 90.54) (layer "F.SilkS")
+  (gr_text "peakick V1\n\nhttps://github.com/rrainey/tempo\nRiley Rainey 2023" (at 130.96 90.54) (layer "F.SilkS")
     (effects (font (size 1 1) (thickness 0.15)) (justify left bottom))
   )

Commit message: Add pull-ups for I2C
Connections:
- net /D5 renamed /D4
- net /D9 renamed /D8
