File: hardware/tempo/tempo.kicad_sch (KiCad schematic)
At the start: 61 parts, among them J3 QWIIC_CONNECTORJS-1MM, J4 10103594-0001LF, J4 3221-10-0300-00-TR, Q1 DMP3125L, SW1 JS102011SAQN, U1 MCP73831, U2 ATSAMD51J20A-A, U2 SAM-M10Q, U3 SPX3819M5-L-3-3/TR, U4 MMC5983MA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

Commit message: renamed new tempo project
Parts:
- D2: MANUFACTURER (none) -> ST Microelectronics; MPN (none) -> BAT20JFILM
- J4: MPN (none) -> 10103594-0001LF

Commit message: updated pcb and enclosure files
Other:
- note added: "SPI Connection - CS = D5"
- note removed: "SPI Connection - CS = D0"
Changed lines of the file:
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@@
     (effects (font (size 2.54 2.54) (thickness 0.508) bold) (justify left bottom))
   )
-  (text "SPI Connection - CS = D0\n" (at 172.72 17.78 0)
+  (text "SPI Connection - CS = D5\n" (at 172.72 17.78 0)
     (effects (font (size 1.27 1.27)) (justify left bottom))
   )
